Commit message: Updated URDF, Added Inertia

File: description/robot_core.xacro (robot description, xacro)
@@ -2,4 +2,5 @@
 <robot xmlns:xacro="http://www.ros.org/wiki/xacro">
     <xacro:include filename="colours.xacro" />
+    <xacro:include filename="inertial_macros.xacro" />
     <!-- BASE LINK -->
     <link name="base_link">
@@ -19,4 +20,13 @@
             <material name ="red"/>
         </visual>
+        <collision>
+            <origin xyz = "0 0 0.15"/>
+            <geometry>
+                <box size = "1 0.7 0.3"/>
+            </geometry>
+        </collision>
+        <xacro:inertial_box mass="1" x="1" y="0.7" z="0.3">
+            <origin xyz="0 0 0.15" rpy="0 0 0"/>
+        </xacro:inertial_box>
     </link>
     <!-- LEFT FRONT WHEEL-->
@@ -34,4 +44,12 @@
             <material name ="white"/>
         </visual>
+        <collision>
+            <geometry>
+                <cylinder radius = "0.15" length="0.1"/>
+            </geometry>
+        </collision>
+        <xacro:inertial_cylinder mass="0.1" length="0.1" radius="0.15">
+            <origin xyz="0 0 0" rpy="0 0 0"/>
+        </xacro:inertial_cylinder>
     </link>
     <!-- RIGHT FRONT WHEEL-->
@@ -49,4 +67,12 @@
             <material name ="white"/>
         </visual>
+        <collision>
+            <geometry>
+                <cylinder radius = "0.15" length="0.1"/>
+            </geometry>
+        </collision>
+        <xacro:inertial_cylinder mass="0.1" length="0.1" radius="0.15">
+            <origin xyz="0 0 0" rpy="0 0 0"/>
+        </xacro:inertial_cylinder>
     </link>
     <!-- LEFT BACK WHEEL-->
@@ -64,4 +90,12 @@
             <material name ="white"/>
         </visual>
+        <collision>
+            <geometry>
+                <cylinder radius = "0.15" length="0.1"/>
+            </geometry>
+        </collision>
+        <xacro:inertial_cylinder mass="0.1" length="0.1" radius="0.15">
+            <origin xyz="0 0 0" rpy="0 0 0"/>
+        </xacro:inertial_cylinder>
     </link>
     <!-- RIGHT BACK WHEEL-->
@@ -79,4 +113,12 @@
             <material name ="white"/>
         </visual>
+        <collision>
+            <geometry>
+                <cylinder radius = "0.15" length="0.1"/>
+            </geometry>
+        </collision>
+        <xacro:inertial_cylinder mass="0.1" length="0.1" radius="0.15">
+            <origin xyz="0 0 0" rpy="0 0 0"/>
+        </xacro:inertial_cylinder>
     </link>
 </robot>

Commit message: Added Gazebo Launch Operation

File: description/robot_core.xacro (robot description, xacro)
@@ -30,4 +30,7 @@
         </xacro:inertial_box>
     </link>
+    <gazebo reference = "chassis_link">
+        <material> Gazebo/Red </material>
+    </gazebo>
     <!-- LEFT FRONT WHEEL-->
     <joint name = "lf_wheel_joint" type= "continuous">
@@ -53,4 +56,7 @@
         </xacro:inertial_cylinder>
     </link>
+    <gazebo reference = "lf_wheel_link">
+        <material> Gazebo/White </material>
+    </gazebo>
     <!-- RIGHT FRONT WHEEL-->
     <joint name = "rf_wheel_joint" type= "continuous">
@@ -76,4 +82,7 @@
         </xacro:inertial_cylinder>
     </link>
+    <gazebo reference = "rf_wheel_link">
+        <material> Gazebo/White </material>
+    </gazebo>
     <!-- LEFT BACK WHEEL-->
     <joint name = "lb_wheel_joint" type= "continuous">
@@ -99,4 +108,7 @@
         </xacro:inertial_cylinder>
     </link>
+    <gazebo reference = "lb_wheel_link">
+        <material> Gazebo/White </material>
+    </gazebo>
     <!-- RIGHT BACK WHEEL-->
     <joint name = "rb_wheel_joint" type= "continuous">
@@ -122,3 +134,6 @@
         </xacro:inertial_cylinder>
     </link>
+    <gazebo reference = "rb_wheel_link">
+        <material> Gazebo/White </material>
+    </gazebo>
 </robot>
